File: Mark2C++.kicad_pcb (KiCad board)
At the start: 2 copper layers, 267 parts, among them U1 12AX7, U10 L7812, U11 6P6S, U15 6P6S, U2 12AX7, U3 12AX7, U4 NE5532, U5 NE5532, U6 NE5532, U7 NE5532, U8 NE5532, U9 LR8

Commit message: changes in schema and pcb
updated schemaitc and pcb
Parts:
- removed 12V_1, 12V_2, 300V_1, 300V_2, 369V1, 369V2, 375V1, 375V2, 385V1, 385V2, 6.3V_1, 6.3V_2, EQ0, EQ1, EQ10, EQ11, EQ20, EQ21, EQ30, EQ31, EQ40, EQ41, EQ50, EQ51, EQ_GND1, EQ_GND2, EQ_IN1, EQ_IN2, EQ_OUT1, EQ_OUT2, FROM_CF1, FROM_EQ1, FROM_FX1, FS_1, FS_2, FX_GND1, FX_GND2, FX_IN1, FX_IN2, FX_IN3, FX_OUT1, FX_OUT2, GND1, GND2, GND3, GRN1, GRN2, HT_1, HT_2, LD0, LD1, LD10, LD11, LD20, LD21, LD30, LD31, LED1, LED2, PA_GND1, PA_IN1, PT1, PT11, PT12, PT2, PT30, PT31, RED1, RED2, RELAY_12V1, RELAY_12V2, RELAY_12V3, RELAY_12V4, RELAY_GND1, RELAY_GND2, RELAY_GND3, RELAY_GND4, TG_3, TG_4, TO_EQ1: Conn_01x01_Female, Connectors:1X01_2MM
- removed 750Hz1, 750Hz2: 50K Lin, Potentiometer_THT:Potentiometer_Bourns_PTA4543_Single_Slide
- removed BRGH_BOOST_C1, BRGH_BOOST_L1, B_Shift1, TREB_SHIFT1: SW_SPDT, Switches:SWITCH_SPDT_PTH_11.6X4.0MM_KIT
- removed D10: RED, LED:LED_5MM
- removed D9: GRN, LED:LED_5MM
- removed EQ_ON/OFF1, FX_ON/OFF1: SWITCH-DPDT-PTH-GPI-152-3013, Switches:SWITCH_DPDT_PTH_GPI-152-3013
- removed U11, U15: 6P6S, Valve:Valve_Octal
- removed U2, U3: 12AX7, Valve:Valve_ECC-83-2
- added 240Hz1: 50K Lin, Potentiometer_THT:Potentiometer_Bourns_PTA4543_Single_Slide, F.Cu at (-204.0, 105.5)
- added 80Hz1: 50K Lin, Potentiometer_THT:Potentiometer_Bourns_PTA4543_Single_Slide, F.Cu at (-204.0, 141.8)
- added C59: 22nF 400V, Capacitor_THT:C_Rect_L18.0mm_W6.0mm_P15.00mm_FKS3_FKP3, F.Cu at (-62.2, 130.6)
- added U12: 6N2P-EW, Valve:Valve_Noval_P, F.Cu at (-105.6, 28.3)
- added U13: 6N2P-EW, Valve:Valve_Noval_P, F.Cu at (-105.6, 52.0)
- added U14: 6N2P-EW, Valve:Valve_Noval_P, F.Cu at (-105.6, 75.7)
- U1: value 12AX7 -> EL34; footprint Valve:Valve_ECC-83-2 -> Valve:Valve_Octal
- moved C11 475.3 mm to (-203.0, 177.1)
- moved U10 429.2 mm to (-155.4, 184.4)
- moved C33 427.0 mm to (-173.9, 183.6)
- moved C24 389.1 mm to (-173.9, 177.1)
- moved C20 382.3 mm to (-182.6, 176.2)
- moved D4 376.3 mm to (-157.0, 175.9)
- moved R8 375.2 mm to (-142.1, 124.7)
- moved R5 374.0 mm to (-142.1, 110.5)
- moved C25 372.4 mm to (-189.4, 185.6)
- moved R4 366.9 mm to (-142.1, 105.7)
- moved C1 361.7 mm to (-82.9, 158.6)
- moved C6 360.9 mm to (-82.9, 176.4)
- moved R41 359.9 mm to (-110.4, 143.7)
- moved R58 359.8 mm to (-94.6, 148.5)
- moved C58 355.6 mm to (-182.6, 185.7)
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Connections:
- C25 pad 1: Net-(C25-Pad1) -> Net-(U12B-K)
- C26 pad 2: Net-(C26-Pad2) -> Net-(U12B-A)
- C3 pad 1: Net-(B_Shift1-Pad2) -> Net-(B_Shift1-B)
- C34 pad 1: Net-(C34-Pad1) -> Net-(U1A-F1)
- C35 pad 2: Net-(C35-Pad2) -> Net-(TG_4-Pin_1)
- C4 pad 1: Net-(B_Shift1-Pad2) -> Net-(B_Shift1-B)
- Inupt1 pad T: Net-(Inupt1-PadT) -> Net-(U12A-G)
- MASTER1 pad 2: Net-(MASTER1-Pad2) -> Net-(U1A-G1)
- R2 pad 1: Net-(Inupt1-PadT) -> Net-(U12A-G)
- R27 pad 1: Net-(C25-Pad1) -> Net-(U12B-K)
- R28 pad 2: Net-(C26-Pad2) -> Net-(U12B-A)
- R3 pad 1: Net-(B_Shift1-Pad2) -> Net-(B_Shift1-B)
- R47 pad 1: Net-(C34-Pad1) -> Net-(U1A-F1)
- R48 pad 2: Net-(R48-Pad2) -> Net-(U1A-G2)
- R5 pad 2: Net-(EQ0-Pad1) -> Net-(EQ0-Pin_1)
- Send1 pad TN: (no net) -> unconnected-(Send1-PadTN)
- U1 pad 1: Net-(C26-Pad2) -> unconnected-(U1A-G3-Pad1)
- U1 pad 2: Net-(EQ30-Pad1) -> unconnected-(U1B-F1-Pad2)
- U1 pad 3: Net-(C25-Pad1) -> Net-(TG_4-Pin_1)
- U1 pad 4: (no net) -> Net-(U1A-G2)
- U1 pad 5: (no net) -> Net-(U1A-G1)
- U1 pad 6: Net-(EQ0-Pad1) -> (no net)
- U1 pad 7: Net-(Inupt1-PadT) -> unconnected-(U1B-F2-Pad7)
- U1 pad 8: Net-(B_Shift1-Pad2) -> Net-(U1A-F1)
- U8 pad 5: (no net) -> unconnected-(U8B-+-Pad5)
Routing:
- net GND: track 50.9 -> 0.00 mm
Other:
- net class Default removed
